Commit message: hopefully everything

File: src/drive/models/drive (1)/urdf/drive.urdf (robot description, URDF)
Before this commit: robot drive3, 13 links, 12 joints
Links:
- removed link steer_1
- removed link steer_2
- removed link steer_3
- removed link steer_4
- removed link steer_5
- removed link steer_6
- added link left_back, mass 0.462954112817127; collision mesh filename=package://drive/meshes/left_back.STL; visual mesh filename=package://drive/meshes/left_back.STL
- added link left_bogie, mass 0.59393; collision mesh filename=package://drive/meshes/left_bogie.STL; visual mesh filename=package://drive/meshes/left_bogie.STL
- added link left_front, mass 0.26897; collision mesh filename=package://drive/meshes/left_front.STL; visual mesh filename=package://drive/meshes/left_front.STL
- added link right_back, mass 0.46295; collision mesh filename=package://drive/meshes/right_back.STL; visual mesh filename=package://drive/meshes/right_back.STL
- added link right_bogie, mass 0.59393; collision mesh filename=package://drive/meshes/right_bogie.STL; visual mesh filename=package://drive/meshes/right_bogie.STL
- added link right_front, mass 0.26897; collision mesh filename=package://drive/meshes/right_front.STL; visual mesh filename=package://drive/meshes/right_front.STL
- link base: mass 18.063 -> 34.1059688345868; geometry collision mesh filename=package://drive/meshes/base.STL; visual mesh filename=package://drive/meshes/base.STL
- link wheel_1: mass 3.55769702765534 -> 32.802; geometry collision mesh filename=package://drive/meshes/wheel_1.STL; visual mesh filename=package://drive/meshes/wheel_1.STL
- link wheel_2: mass 3.55819809981133 -> 32.802; geometry collision mesh filename=package://drive/meshes/wheel_2.STL; visual mesh filename=package://drive/meshes/wheel_2.STL
- link wheel_3: mass 3.55769708838011 -> 32.802; geometry collision mesh filename=package://drive/meshes/wheel_3.STL; visual mesh filename=package://drive/meshes/wheel_3.STL
- link wheel_4: mass 3.55826837186396 -> 32.802; geometry collision mesh filename=package://drive/meshes/wheel_4.STL; visual mesh filename=package://drive/meshes/wheel_4.STL
- link wheel_5: mass 3.55769706915786 -> 32.802; geometry collision mesh filename=package://drive/meshes/wheel_5.STL; visual mesh filename=package://drive/meshes/wheel_5.STL
- link wheel_6: mass 3.55826721651292 -> 32.8019150211691; geometry collision mesh filename=package://drive/meshes/wheel_6.STL; visual mesh filename=package://drive/meshes/wheel_6.STL
Joints:
- removed joint steer_joint_1
- removed joint steer_joint_2
- removed joint steer_joint_3
- removed joint steer_joint_4
- removed joint steer_joint_5
- removed joint steer_joint_6
- removed joint wheel_joint_1
- removed joint wheel_joint_2
- removed joint wheel_joint_3
- removed joint wheel_joint_4
- removed joint wheel_joint_5
- removed joint wheel_joint_6
- added joint joint_left_back: type revolute, parent base, child left_back, origin xyz=-0.54534 -0.10578 -0.012427 rpy=-1.5708 0.12123 1.5708, axis 0 0 1, limit lower=0 upper=0 effort=0 velocity=0
- added joint joint_left_bogie: type revolute, parent left_front, child left_bogie, origin xyz=-0.31109 -0.16078 0 rpy=0 0 -0.12123, axis 0 0 1, limit lower=0 upper=0 effort=0 velocity=0
- added joint joint_left_front: type revolute, parent base, child left_front, origin xyz=-0.56534 -0.15578 -0.062427 rpy=-1.5708 0.12123 1.5708, axis 0 0 1, limit lower=0 upper=0 effort=0 velocity=0
- added joint joint_right_back: type revolute, parent base, child right_back, origin xyz=0 -0.10542 -0.012427 rpy=-1.5708 0.12123 1.5708, axis 0 0 1, limit lower=0 upper=0 effort=0 velocity=0
- added joint joint_right_bogie: type revolute, parent right_front, child right_bogie, origin xyz=-0.31109 -0.16078 0 rpy=-3.1416 0 3.0204, axis 0 0 1, limit lower=0 upper=0 effort=0 velocity=0
- added joint joint_right_front: type revolute, parent base, child right_front, origin xyz=-0.070337 -0.15542 -0.062427 rpy=-1.5708 0.12123 1.5708, axis 0 0 1, limit lower=0 upper=0 effort=0 velocity=0
- added joint joint_wheel_1: type revolute, parent right_bogie, child wheel_1, origin xyz=0.225 -0.18509 0 rpy=0.16161 1.4835 0.35684, axis 0.99619 -0.014024 -0.08602, limit lower=0 upper=0 effort=0 velocity=0
- added joint joint_wheel_2: type revolute, parent right_bogie, child wheel_2, origin xyz=-0.225 -0.18509 0 rpy=0.16161 1.4835 0.42392, axis 0.99619 -0.014024 -0.08602, limit lower=0 upper=0 effort=0 velocity=0
- added joint joint_wheel_3: type revolute, parent right_back, child wheel_3, origin xyz=0.45337 -0.39 0 rpy=-2.98 -1.4835 2.1495, axis 0.99619 -0.014024 -0.08602, limit lower=0 upper=0 effort=0 velocity=0
- added joint joint_wheel_4: type revolute, parent left_bogie, child wheel_4, origin xyz=-0.225 -0.18509 0.016876 rpy=0.16161 1.4835 -0.33202, axis 0.99619 -0.014024 -0.08602, limit lower=0 upper=0 effort=0 velocity=0
- added joint joint_wheel_5: type revolute, parent left_bogie, child wheel_5, origin xyz=0.225 -0.18509 0.016876 rpy=0.16161 1.4835 -1.252, axis 0.99619 -0.014024 -0.08602, limit lower=0 upper=0 effort=0 velocity=0
- added joint joint_wheel_6: type revolute, parent left_back, child wheel_6, origin xyz=0.45337 -0.39 0.034376 rpy=0.16161 1.4835 -0.74019, axis 0.99619 -0.014024 -0.08602, limit lower=0 upper=0 effort=0 velocity=0
