Commit message: World development and sensor addition

File: src/drive/models/drive/urdf/drive.urdf (robot description, URDF)
Before this commit: robot drive, 13 links, 12 joints
Links:
- removed link base
- added link base_link, mass 12.6951056650873; collision mesh filename=package://drive/meshes/base.STL; visual mesh filename=package://drive/meshes/base.STL
- added link imu_link
- added link lidar_link
Joints:
- added joint imu_joint: type fixed, parent base_link, child imu_link
- added joint lidar_joint: type fixed, parent base_link, child lidar_link
- joint joint_rotate_1: parent base -> base_link
- joint joint_rotate_2: parent base -> base_link
- joint joint_rotate_3: parent base -> base_link
- joint joint_rotate_4: parent base -> base_link
- joint joint_rotate_5: parent base -> base_link
- joint joint_rotate_6: parent base -> base_link

Commit message: topic fix

File: src/drive/models/drive/urdf/drive.urdf (robot description, URDF)
Before this commit: robot drive, 15 links, 14 joints
Links:
- link imu_link: mass None -> 0.01; geometry collision box ; visual box 
- link lidar_link: mass None -> 0.01; geometry collision cylinder ; visual cylinder 

Commit message: ros2 control

File: src/drive/models/drive/urdf/drive.urdf (robot description, URDF)
Before this commit: robot drive, 15 links, 14 joints
Joints:
- joint joint_rotate_5: axis 0 0.6257 0.78007 -> 0 0 1
- joint joint_rotate_6: axis 0 0.075039 -0.99718 -> 0 0 1

Commit message: sensors fix

File: src/drive/models/drive/urdf/drive.urdf (robot description, URDF)
Before this commit: robot drive, 15 links, 14 joints
Links:
- link imu_link: geometry collision box size=0.01 0.01 0.01; visual box size=0.01 0.01 0.01
- link lidar_link: geometry collision cylinder length=0.02 radius=0.03; visual cylinder length=0.02 radius=0.03
Joints:
- joint imu_joint: origin (none) -> xyz=0 0 0.1 rpy=0 0 0
- joint lidar_joint: origin (none) -> xyz=0 0 0.2 rpy=0 0 0

Commit message: New Rover

File: src/drive/models/drive/urdf/drive.urdf (robot description, URDF)
Before this commit: robot drive, 15 links, 14 joints
Links:
- removed link base_link
- removed link imu_link
- removed link lidar_link
- removed link rotate_1
- removed link rotate_2
- removed link rotate_3
- removed link rotate_4
- removed link rotate_5
- removed link rotate_6
- added link base, mass 34.1059688345868; collision mesh filename=package://drive/meshes/base.STL; visual mesh filename=package://drive/meshes/base.STL
- added link left_back, mass 0.462954112817127; collision mesh filename=package://drive/meshes/left_back.STL; visual mesh filename=package://drive/meshes/left_back.STL
- added link left_bogie, mass 0.59393; collision mesh filename=package://drive/meshes/left_bogie.STL; visual mesh filename=package://drive/meshes/left_bogie.STL
- added link left_front, mass 0.26897; collision mesh filename=package://drive/meshes/left_front.STL; visual mesh filename=package://drive/meshes/left_front.STL
- added link right_back, mass 0.46295; collision mesh filename=package://drive/meshes/right_back.STL; visual mesh filename=package://drive/meshes/right_back.STL
- added link right_bogie, mass 0.59393; collision mesh filename=package://drive/meshes/right_bogie.STL; visual mesh filename=package://drive/meshes/right_bogie.STL
- added link right_front, mass 0.26897; collision mesh filename=package://drive/meshes/right_front.STL; visual mesh filename=package://drive/meshes/right_front.STL
- link wheel_1: mass 0.969966731795849 -> 32.802
- link wheel_2: mass 0.969966731795848 -> 32.802
- link wheel_3: mass 0.969966731795848 -> 32.802
- link wheel_4: mass 0.969966731795849 -> 32.802
- link wheel_5: mass 0.969966731795849 -> 32.802
- link wheel_6: mass 0.969966731795848 -> 32.8019150211691
Joints:
- removed joint imu_joint
- removed joint joint_rotate_1
- removed joint joint_rotate_2
- removed joint joint_rotate_3
- removed joint joint_rotate_4
- removed joint joint_rotate_5
- removed joint joint_rotate_6
- removed joint lidar_joint
- added joint joint_left_back: type revolute, parent base, child left_back, origin xyz=-0.54534 -0.10578 -0.012427 rpy=-1.5708 0.12123 1.5708, axis 0 0 1, limit lower=-1.0 upper=1.0 effort=10 velocity=0
- added joint joint_left_bogie: type revolute, parent left_front, child left_bogie, origin xyz=-0.31109 -0.16078 0 rpy=0 0 -0.12123, axis 0 0 1, limit lower=-3.14159 upper=3.14159 effort=10 velocity=0
- added joint joint_left_front: type revolute, parent base, child left_front, origin xyz=-0.56534 -0.15578 -0.062427 rpy=-1.5708 0.12123 1.5708, axis 0 0 1, limit lower=-1.0 upper=1.0 effort=10 velocity=0
- added joint joint_right_back: type revolute, parent base, child right_back, origin xyz=0 -0.10542 -0.012427 rpy=-1.5708 0.12123 1.5708, axis 0 0 1, limit lower=-1.0 upper=1.0 effort=10 velocity=0
- added joint joint_right_bogie: type revolute, parent right_front, child right_bogie, origin xyz=-0.31109 -0.16078 0 rpy=-3.1416 0 3.0204, axis 0 0 1, limit lower=-3.14159 upper=3.14159 effort=10 velocity=0
- added joint joint_right_front: type revolute, parent base, child right_front, origin xyz=-0.070337 -0.15542 -0.062427 rpy=-1.5708 0.12123 1.5708, axis 0 0 1, limit lower=-1.0 upper=1.0 effort=10 velocity=0
- joint joint_wheel_1: axis 0 1 0 -> 1 0 0; origin xyz=0 0 0.1125 rpy=3.1416 1.3751 1.5708 -> xyz=0.225 -0.18509 0 rpy=-1.5707 1.5707 0; parent rotate_1 -> right_bogie
- joint joint_wheel_2: axis 0 1 0 -> 1 0 0; origin xyz=0 0 0.1125 rpy=0 0.1965 -1.5708 -> xyz=-0.225 -0.18509 0 rpy=-1.5707 1.5707 0; parent rotate_2 -> right_bogie
- joint joint_wheel_3: axis 0 1 0 -> 1 0 0; origin xyz=0 0 0.11241 rpy=0 0.67825 1.5708 -> xyz=0.45337 -0.39 0 rpy=-1.5707 1.5707 0; parent rotate_3 -> right_back
- joint joint_wheel_4: axis 0 1 0 -> 1 0 0; origin xyz=0 0 0.1125 rpy=0 0.6986 -1.5708 -> xyz=-0.225 -0.18509 0.016876 rpy=-1.5707 1.5707 0; parent rotate_4 -> left_bogie
- joint joint_wheel_5: axis 0 1 0 -> 1 0 0; origin xyz=0 0.070391 0.087757 rpy=0 0.025369 -1.5708 -> xyz=0.225 -0.18509 0.016876 rpy=-1.5707 1.5707 0; parent rotate_5 -> left_bogie
- joint joint_wheel_6: axis 0 1 0 -> 1 0 0; origin xyz=0 -0.0084274 0.11199 rpy=3.1416 -0.69655 -1.5708 -> xyz=0.45337 -0.39 0.034376 rpy=-1.5707 1.5707 0; parent rotate_6 -> left_back

Commit message: sensors

File: src/drive/models/drive/urdf/drive.urdf (robot description, URDF)
Before this commit: robot drive, 13 links, 12 joints
Links:
- added link imu_link, mass 0.01; collision box size=0.01 0.01 0.01; visual box size=0.01 0.01 0.01
- added link lidar_link, mass 0.01; collision cylinder length=0.02 radius=0.03; visual cylinder length=0.02 radius=0.03
Joints:
- added joint imu_joint: type fixed, parent base, child imu_link, origin xyz=0 0 0.1 rpy=0 0 0
- added joint lidar_joint: type fixed, parent base, child lidar_link, origin xyz=0 0 0.2 rpy=0 0 0

Commit message: sensor positions

File: src/drive/models/drive/urdf/drive.urdf (robot description, URDF)
Before this commit: robot drive, 15 links, 14 joints
Joints:
- joint imu_joint: origin xyz=0 0 0.1 rpy=0 0 0 -> xyz=-0.345788930637997 -0.153460943930369 0.05 rpy=0 0 0
- joint lidar_joint: origin xyz=0 0 0.2 rpy=0 0 0 -> xyz=-0.345788930637997 -0.153460943930369 -0.12 rpy=0 0 0

Commit message: new_unfixed_urdf

File: src/drive/models/drive/urdf/drive.urdf (robot description, URDF)
Before this commit: robot drive, 15 links, 14 joints
Links:
- removed link left_back
- removed link left_bogie
- removed link left_front
- removed link right_back
- removed link right_bogie
- removed link right_front
- link base: mass 34.1059688345868 -> 36.758
- link wheel_6: mass 32.8019150211691 -> 32.802
Joints:
- removed joint joint_left_back
- removed joint joint_left_bogie
- removed joint joint_left_front
- removed joint joint_right_back
- removed joint joint_right_bogie
- removed joint joint_right_front
- removed joint joint_wheel_1
- removed joint joint_wheel_2
- removed joint joint_wheel_3
- removed joint joint_wheel_4
- removed joint joint_wheel_5
- removed joint joint_wheel_6
- added joint wheel_joint_1: type continuous, parent base, child wheel_1, origin xyz=-0.12406 -0.94233 0.11392 rpy=1.0129 -0.057594 3.076, axis 0.99619 -0.014024 -0.08602
- added joint wheel_joint_2: type continuous, parent base, child wheel_2, origin xyz=0.36212 -0.94269 0.11392 rpy=1.71 -0.0019564 -0.087245, axis 0.99619 -0.014024 -0.08602
- added joint wheel_joint_3: type continuous, parent base, child wheel_3, origin xyz=-0.12406 -0.49233 0.11392 rpy=0.83798 -0.068122 3.087, axis 0.99619 -0.014024 -0.08602
- added joint wheel_joint_4: type continuous, parent base, child wheel_4, origin xyz=0.36212 -0.49269 0.11392 rpy=1.9152 0.015899 -0.08581, axis 0.99619 -0.014024 -0.08602
- added joint wheel_joint_5: type continuous, parent base, child wheel_5, origin xyz=-0.12156 0.11889 0.11392 rpy=0.12629 -0.087212 -3.1385, axis 0.99619 -0.014024 -0.08602
- added joint wheel_joint_6: type continuous, parent base, child wheel_6, origin xyz=0.35962 0.11889 0.11392 rpy=1.9946 0.022675 -0.084276, axis 0.99619 -0.014024 -0.08602
- joint imu_joint: origin xyz=-0.345788930637997 -0.153460943930369 0.05 rpy=0 0 0 -> xyz=0.0 0.0 0.1 rpy=0 0 0
- joint lidar_joint: origin xyz=-0.345788930637997 -0.153460943930369 -0.12 rpy=0 0 0 -> xyz=0.0 0.0 0.15 rpy=0 0 0

File: src/sam_bot_nav2_gz/src/description/sam_bot_description.urdf (robot description, URDF)
Before this commit: robot sam_bot, 7 links, 6 joints
Joints:
- joint base_joint: child base_footprint -> base_link; origin xyz=0.0 0.0 ${-(wheel_radius+wheel_zoff)} rpy=0 0 0 -> xyz=0.0 0.0 ${(wheel_radius+wheel_zoff)} rpy=0 0 0; parent base_link -> base_footprint

Commit message: zed2+lidar+imu

File: src/drive/models/drive/urdf/drive.urdf (robot description, URDF)
Before this commit: robot drive, 9 links, 8 joints
Links:
- added link ZED_camera_link, mass 0.2; collision mesh filename=package://drive/meshes/zed2i.stl scale=1 1 1; visual mesh filename=package://drive/meshes/zed2i.stl scale=1 1 1
- added link ZED_center_camera_frame
- added link ZED_center_camera_frame_sensor, mass 0.0001
- added link ZED_center_camera_optical
- added link ZED_left_camera_frame
- added link ZED_left_camera_frame_sensor, mass 0.0001
- added link ZED_left_camera_optical
- added link ZED_right_camera_frame
- added link ZED_right_camera_frame_sensor, mass 0.0001
- added link ZED_right_camera_optical
- added link base_link
- link imu_link: geometry collision box size=1 1 1; visual box size=0.01 0.01 0.01
- link lidar_link: geometry visual cylinder length=5 radius=3
Joints:
- added joint ZED_center_camera_joint: type fixed, parent ZED_camera_link, child ZED_center_camera_frame, origin xyz=0 0 0 rpy=0 0 0
- added joint ZED_center_camera_optical_joint: type fixed, parent ZED_center_camera_frame, child ZED_center_camera_optical, origin xyz=0 0 0 rpy=-1.5708 0 -1.5708
- added joint ZED_center_camera_sensor_joint: type fixed, parent ZED_center_camera_frame, child ZED_center_camera_frame_sensor, origin xyz=0 0 0 rpy=0 0 0
- added joint ZED_joint: type fixed, parent base, child ZED_camera_link, origin xyz=0.12 0.0 0.25 rpy=0 0 0
- added joint ZED_left_camera_joint: type fixed, parent ZED_camera_link, child ZED_left_camera_frame, origin xyz=0 0.06 0 rpy=0 0 0
- added joint ZED_left_camera_optical_joint: type fixed, parent ZED_left_camera_frame, child ZED_left_camera_optical, origin xyz=0 0 0 rpy=-1.5708 0 -1.5708
- added joint ZED_left_camera_sensor_joint: type fixed, parent ZED_left_camera_frame, child ZED_left_camera_frame_sensor, origin xyz=0 0 0 rpy=0 0 0
- added joint ZED_right_camera_joint: type fixed, parent ZED_camera_link, child ZED_right_camera_frame, origin xyz=0 -0.06 0 rpy=0 0 0
- added joint ZED_right_camera_optical_joint: type fixed, parent ZED_right_camera_frame, child ZED_right_camera_optical, origin xyz=0 0 0 rpy=-1.5708 0 -1.5708
- added joint ZED_right_camera_sensor_joint: type fixed, parent ZED_right_camera_frame, child ZED_right_camera_frame_sensor, origin xyz=0 0 0 rpy=0 0 0
- added joint base_joint: type fixed, parent base_link, child base
- joint imu_joint: origin xyz=0.0 0.0 0.1 rpy=0 0 0 -> xyz=0.5 -0.2 .5 rpy=0 0 0
- joint lidar_joint: origin xyz=0.0 0.0 0.15 rpy=0 0 0 -> xyz=0.3 0 0.5 rpy=0 0 0
- joint wheel_joint_1: origin xyz=-0.12406 -0.94233 0.11392 rpy=1.0129 -0.057594 3.076 -> xyz=-0.12406 -0.94233 -0.11392 rpy=1.0129 -0.057594 3.076
- joint wheel_joint_2: origin xyz=0.36212 -0.94269 0.11392 rpy=1.71 -0.0019564 -0.087245 -> xyz=0.36212 -0.94269 -0.11392 rpy=1.71 -0.0019564 -0.087245
- joint wheel_joint_3: origin xyz=-0.12406 -0.49233 0.11392 rpy=0.83798 -0.068122 3.087 -> xyz=-0.12406 -0.49233 -0.11392 rpy=0.83798 -0.068122 3.087
- joint wheel_joint_4: origin xyz=0.36212 -0.49269 0.11392 rpy=1.9152 0.015899 -0.08581 -> xyz=0.36212 -0.49269 -0.11392 rpy=1.9152 0.015899 -0.08581
- joint wheel_joint_5: origin xyz=-0.12156 0.11889 0.11392 rpy=0.12629 -0.087212 -3.1385 -> xyz=-0.12156 0.11889 -0.11392 rpy=0.12629 -0.087212 -3.1385
- joint wheel_joint_6: origin xyz=0.35962 0.11889 0.11392 rpy=1.9946 0.022675 -0.084276 -> xyz=0.35962 0.11889 -0.11392 rpy=1.9946 0.022675 -0.084276

Commit message: imu_working

File: src/drive/models/drive/urdf/drive.urdf (robot description, URDF)
Before this commit: robot drive, 20 links, 19 joints
Links:
- link lidar_link: geometry visual cylinder length=0.05 radius=0.03

Commit message: xacro

File: src/drive/models/drive/urdf/drive.urdf (robot description, URDF)
Before this commit: robot drive, 15 links, 14 joints
Links:
- removed link lidar_link
- link imu_link: geometry collision box size=1 1 1; visual box size=0.01 0.01 0.01
Joints:
- removed joint lidar_joint
- joint imu_joint: origin xyz=-0.345788930637997 -0.153460943930369 0.05 rpy=0 0 0 -> xyz=0.5 -0.2 .5 rpy=0 0 0
- joint joint_left_back: type revolute -> fixed
- joint joint_right_back: type revolute -> fixed
- joint joint_right_bogie: type revolute -> fixed
- joint joint_right_front: type revolute -> fixed

Commit message: depth testing

File: src/drive/models/drive/urdf/drive.urdf (robot description, URDF)
Before this commit: robot drive, 13 links, 12 joints
Links:
- added link depth_camera_link; visual box 
Joints:
- added joint depth_camera_joint: type fixed, parent base, child depth_camera_link, origin xyz=0.2 0 0.3 rpy=0 0 0

Commit message: fixed orientation but lidar not working and clock

File: src/drive/models/drive/urdf/drive.urdf (robot description, URDF)
Before this commit: robot drive, 15 links, 14 joints
Links:
- added link base_link
Joints:
- added joint base_joint: type fixed, parent base_link, child base, origin xyz=0 0 0 rpy=0 -3.1415 0
- joint imu_joint: parent base -> base_link
- joint lidar_joint: parent base -> base_link

Commit message: position of sensors

File: src/drive/models/drive/urdf/drive.urdf (robot description, URDF)
Before this commit: robot drive, 16 links, 15 joints
Joints:
- joint imu_joint: origin xyz=-0.345788930637997 -0.153460943930369 0.05 rpy=0 0 0 -> xyz=0.45 -0.3 0.05 rpy=0 0 0
- joint lidar_joint: origin xyz=-0.345788930637997 -0.153460943930369 -0.12 rpy=0 0 0 -> xyz=0.45 -0.3 0.12 rpy=0 0 0

Commit message: lidar position fixed

File: src/drive/models/drive/urdf/drive.urdf (robot description, URDF)
Before this commit: robot drive, 16 links, 15 joints
Joints:
- joint lidar_joint: origin xyz=0.45 -0.3 0.12 rpy=0 0 0 -> xyz=0.36 -0.3 0.14 rpy=0 0 0
